Commit message: V2: verify moving Gazebo lidar localization

File: src/aris_description/urdf/aris.urdf.xacro (robot description, xacro)
@@ -11,4 +11,9 @@
   <xacro:property name="max_steer" value="0.6"/>    <!-- rad, steering limit -->
   <xacro:property name="track" value="0.9"/>        <!-- m, approximate wheel track -->
+  <xacro:property name="body_length" value="${wheelbase + 0.4}"/>
+  <xacro:property name="body_width" value="${track}"/>
+  <xacro:property name="body_height" value="0.4"/>
+  <xacro:property name="body_mass" value="80.0"/>
+  <xacro:property name="sensor_mass" value="0.5"/>
   <!-- Injects simulation-only additions (Gazebo sensor plugins) without touching
        the kinematics/TF that the real vehicle also relies on. -->
@@ -16,19 +21,40 @@
   <material name="aris_body"><color rgba="0.15 0.18 0.22 1.0"/></material>
   <material name="aris_sensor"><color rgba="0.85 0.40 0.15 1.0"/></material>
+  <xacro:macro name="box_inertial" params="mass x y z">
+    <inertial>
+      <mass value="${mass}"/>
+      <inertia
+        ixx="${mass * (y * y + z * z) / 12.0}"
+        ixy="0.0"
+        ixz="0.0"
+        iyy="${mass * (x * x + z * z) / 12.0}"
+        iyz="0.0"
+        izz="${mass * (x * x + y * y) / 12.0}"/>
+    </inertial>
+  </xacro:macro>
   <!-- Vehicle base frame: origin at the rear axle on the ground plane. -->
   <link name="base_link">
+    <xacro:box_inertial mass="${body_mass}" x="${body_length}" y="${body_width}" z="${body_height}"/>
     <visual>
       <origin xyz="${wheelbase/2} 0 0.25" rpy="0 0 0"/>
-      <geometry><box size="${wheelbase + 0.4} ${track} 0.4"/></geometry>
+      <geometry><box size="${body_length} ${body_width} ${body_height}"/></geometry>
       <material name="aris_body"/>
     </visual>
+    <collision>
+      <origin xyz="${wheelbase/2} 0 0.25" rpy="0 0 0"/>
+      <geometry><box size="${body_length} ${body_width} ${body_height}"/></geometry>
+    </collision>
   </link>
   <!-- Fixed sensor frame with a small visual marker. -->
   <xacro:macro name="sensor_frame" params="name xyz rpy">
     <link name="${name}">
+      <xacro:box_inertial mass="${sensor_mass}" x="0.08" y="0.08" z="0.08"/>
       <visual>
         <geometry><box size="0.08 0.08 0.08"/></geometry>
         <material name="aris_sensor"/>
       </visual>
+      <collision>
+        <geometry><box size="0.08 0.08 0.08"/></geometry>
+      </collision>
     </link>
     <joint name="${name}_joint" type="fixed">

Commit message: v0: sync headless simulation embedded

File: src/aris_description/urdf/aris.urdf.xacro (robot description, xacro)
@@ -16,4 +16,9 @@
   <xacro:property name="body_mass" value="80.0"/>
   <xacro:property name="sensor_mass" value="0.5"/>
+  <xacro:property name="wheel_radius" value="0.18"/>
+  <xacro:property name="wheel_width" value="0.12"/>
+  <xacro:property name="wheel_mass" value="2.0"/>
+  <xacro:property name="wheel_center_z" value="${wheel_radius + 0.05}"/>
+  <xacro:property name="body_center_z" value="${wheel_center_z + body_height / 2.0}"/>
   <!-- Injects simulation-only additions (Gazebo sensor plugins) without touching
        the kinematics/TF that the real vehicle also relies on. -->
@@ -33,14 +38,26 @@
     </inertial>
   </xacro:macro>
+  <xacro:macro name="wheel_inertial" params="mass radius width">
+    <inertial>
+      <mass value="${mass}"/>
+      <inertia
+        ixx="${mass * (3.0 * radius * radius + width * width) / 12.0}"
+        ixy="0.0"
+        ixz="0.0"
+        iyy="${mass * radius * radius / 2.0}"
+        iyz="0.0"
+        izz="${mass * (3.0 * radius * radius + width * width) / 12.0}"/>
+    </inertial>
+  </xacro:macro>
   <!-- Vehicle base frame: origin at the rear axle on the ground plane. -->
   <link name="base_link">
     <xacro:box_inertial mass="${body_mass}" x="${body_length}" y="${body_width}" z="${body_height}"/>
     <visual>
-      <origin xyz="${wheelbase/2} 0 0.25" rpy="0 0 0"/>
+      <origin xyz="${wheelbase/2} 0 ${body_center_z}" rpy="0 0 0"/>
       <geometry><box size="${body_length} ${body_width} ${body_height}"/></geometry>
       <material name="aris_body"/>
     </visual>
     <collision>
-      <origin xyz="${wheelbase/2} 0 0.25" rpy="0 0 0"/>
+      <origin xyz="${wheelbase/2} 0 ${body_center_z}" rpy="0 0 0"/>
       <geometry><box size="${body_length} ${body_width} ${body_height}"/></geometry>
     </collision>
@@ -76,4 +93,53 @@
   <xacro:sensor_frame name="camera_rear_link"  xyz="-0.4 0 0.7"    rpy="0 0 3.142"/>
   <xacro:if value="$(arg use_sim)">
+    <xacro:macro name="wheel_link" params="name">
+      <link name="${name}">
+        <xacro:wheel_inertial mass="${wheel_mass}" radius="${wheel_radius}" width="${wheel_width}"/>
+        <visual>
+          <origin xyz="0 0 0" rpy="1.57079632679 0 0"/>
+          <geometry><cylinder radius="${wheel_radius}" length="${wheel_width}"/></geometry>
+          <material name="aris_body"/>
+        </visual>
+        <collision>
+          <origin xyz="0 0 0" rpy="1.57079632679 0 0"/>
+          <geometry><cylinder radius="${wheel_radius}" length="${wheel_width}"/></geometry>
+        </collision>
+      </link>
+    </xacro:macro>
+    <xacro:macro name="rear_wheel" params="prefix y">
+      <xacro:wheel_link name="${prefix}_wheel_link"/>
+      <joint name="${prefix}_wheel_joint" type="continuous">
+        <parent link="base_link"/>
+        <child link="${prefix}_wheel_link"/>
+        <origin xyz="0 ${y} ${wheel_center_z}" rpy="0 0 0"/>
+        <axis xyz="0 1 0"/>
+        <dynamics damping="0.05" friction="0.0"/>
+      </joint>
+    </xacro:macro>
+    <xacro:macro name="front_wheel" params="prefix y">
+      <link name="${prefix}_steer_link">
+        <xacro:box_inertial mass="0.2" x="0.04" y="0.04" z="0.04"/>
+      </link>
+      <joint name="${prefix}_steer_joint" type="revolute">
+        <parent link="base_link"/>
+        <child link="${prefix}_steer_link"/>
+        <origin xyz="${wheelbase} ${y} ${wheel_center_z}" rpy="0 0 0"/>
+        <axis xyz="0 0 1"/>
+        <limit lower="${-max_steer}" upper="${max_steer}" effort="100.0" velocity="2.0"/>
+        <dynamics damping="0.2" friction="0.0"/>
+      </joint>
+      <xacro:wheel_link name="${prefix}_wheel_link"/>
+      <joint name="${prefix}_wheel_joint" type="continuous">
+        <parent link="${prefix}_steer_link"/>
+        <child link="${prefix}_wheel_link"/>
+        <origin xyz="0 0 0" rpy="0 0 0"/>
+        <axis xyz="0 1 0"/>
+        <dynamics damping="0.05" friction="0.0"/>
+      </joint>
+    </xacro:macro>
+    <xacro:rear_wheel prefix="rear_left" y="${track / 2.0}"/>
+    <xacro:rear_wheel prefix="rear_right" y="${-track / 2.0}"/>
+    <xacro:front_wheel prefix="front_left" y="${track / 2.0}"/>
+    <xacro:front_wheel prefix="front_right" y="${-track / 2.0}"/>
     <gazebo reference="lidar_link">
       <sensor name="gpu_lidar" type="gpu_lidar">
@@ -105,4 +171,23 @@
       </sensor>
     </gazebo>
+    <gazebo>
+      <plugin filename="gz-sim-ackermann-steering-system" name="gz::sim::systems::AckermannSteering">
+        <left_joint>rear_left_wheel_joint</left_joint>
+        <right_joint>rear_right_wheel_joint</right_joint>
+        <left_steering_joint>front_left_steer_joint</left_steering_joint>
+        <right_steering_joint>front_right_steer_joint</right_steering_joint>
+        <wheel_base>${wheelbase}</wheel_base>
+        <wheel_separation>${track}</wheel_separation>
+        <kingpin_width>${track}</kingpin_width>
+        <wheel_radius>${wheel_radius}</wheel_radius>
+        <steering_limit>${max_steer}</steering_limit>
+        <topic>/cmd_vel</topic>
+        <odom_topic>/gazebo/odom</odom_topic>
+        <tf_topic>/gazebo/tf</tf_topic>
+        <frame_id>odom</frame_id>
+        <child_frame_id>base_link</child_frame_id>
+        <odom_publish_frequency>30</odom_publish_frequency>
+      </plugin>
+    </gazebo>
   </xacro:if>
 </robot>
